File: Akashi-11.kicad_pcb (KiCad board)
At the start: 2 copper layers, 69.9 x 74.9 mm, 43 parts, among them CN10 PPPC192LFBN-RC, CN7 PPPC192LFBN-RC, J1 Conn_02x20_Odd_Even, SW1 SW, U1 MAX6934AQH+D, U2 MAX4719EUB+, U3 TPS613221ADBV, U4 TLV61046ADB

Commit message: Add current measurment point
Parts:
- added JP3: Jumper_2_Open, Connector_PinHeader_2.54mm:PinHeader_1x02_P2.54mm_Vertical, F.Cu at (165.7, 48.3)
- added JP4: SolderJumper_2_Bridged, Jumper:SolderJumper-2_P1.3mm_Bridged_RoundedPad1.0x1.5mm, F.Cu at (170.2, 47.0)
Connections:
- J1 pad 38: +BATT -> Net-(J1-Pad38)
Routing:
- net Net-(J1-Pad38): track 0.00 -> 18.9 mm
- net +BATT: track 53.2 -> 42.7 mm
Other:
- board text added: "Current"

Commit message: Changed from Nucleo to RPi Pico
Parts:
- removed CN10, CN7: PPPC192LFBN-RC, Connector_PinSocket_2.54mm:PinSocket_2x19_P2.54mm_Vertical
- removed R1: 1k, Capacitor_SMD:C_0603_1608Metric_Pad1.08x0.95mm_HandSolder
- added U5: Pico, LOCAL_LIB:RPi_Pico_SMD_TH, F.Cu at (195.6, 67.3)
- D1, D2: footprint Capacitor_SMD:C_0603_1608Metric_Pad1.08x0.95mm_HandSolder -> Diode_SMD:D_0603_1608Metric_Pad1.05x0.95mm_HandSolder
- D3: value LED -> D_Schottky; footprint LED_THT:LED_D4.0mm -> Diode_SMD:D_0603_1608Metric_Pad1.05x0.95mm_HandSolder
- SW1: value SW -> SW_MEC_5E
- moved SW1 83.5 mm to (178.4, 99.3)
- moved TP3 77.6 mm to (123.2, 95.2)
- moved J1 49.7 mm to (167.6, 57.1), turned to 0 degrees
- moved TP6 37.1 mm to (199.4, 101.6)
- moved C1 25.4 mm to (149.9, 54.6), turned to 180 degrees
- moved L1 24.4 mm to (152.6, 48.3)
- moved TP9 23.2 mm to (123.2, 86.4)
- moved TP4 21.8 mm to (123.2, 74.9)
- moved JP4 20.7 mm to (156.2, 62.2)
- moved JP3 20.3 mm to (152.4, 63.5)
- moved JP1 16.2 mm to (160.0, 54.6)
- moved TP5 15.5 mm to (191.8, 101.6)
- moved U3 15.5 mm to (160.0, 50.8)
- moved C6 15.4 mm to (167.6, 47.0), turned to 90 degrees
- moved JP2 14.7 mm to (137.2, 62.2)
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Connections:
- net /SPI1_MOSI renamed /MOSI
- net /SPI1_SCK renamed /SCK
- net /TIM1_CH1 renamed /H_PWM_P
- net /TIM1_CH1N renamed /H_PWM_N
- net /TIM2_CH1 renamed /CHARGE_P_PWM
- D3 pad 2: /STATUS -> +BATT
- SW1 pad 1: GND -> Net-(SW1-Pad1)
- SW1 pad 2: GND -> Net-(SW1-Pad1)
- SW1 pad 3: Net-(CN7-Pad14) -> GND
- SW1 pad 4: Net-(CN7-Pad14) -> GND
- U1 pad 20: /Seg_a -> unconnected-(U1-Pad20)
- U1 pad 25: /D8 -> /D0
- U1 pad 26: /Seg_g -> /Seg_b
- U1 pad 27: /D7 -> /D1
- U1 pad 3: unconnected-(U1-Pad3) -> /Seg_a
- U1 pad 30: /Seg_f -> /D2
- U1 pad 32: /Seg_e -> /DP
- U1 pad 33: /D5 -> /D3
- U1 pad 34: /D4 -> /Seg_d
- U1 pad 35: /Seg_d -> /D4
- U1 pad 36: /D3 -> /D5
- U1 pad 37: /DP -> /Seg_e
- U1 pad 38: /D2 -> /Seg_c
- U1 pad 39: /Seg_c -> /Seg_f
- U1 pad 40: /D1 -> /D7
- U1 pad 41: /Seg_b -> /Seg_g
- U1 pad 42: /D0 -> /D8
Routing:
- net /CHARGE_P_PWM: track 62.1 -> 0.00 mm
- net /SCK: track 52.2 -> 0.00 mm
- net /H_PWM_P: track 47.8 -> 0.00 mm
- net /LOAD: track 46.9 -> 0.00 mm
- net +BATT: track 42.7 -> 0.00 mm
- net /Seg_a: track 41.4 -> 0.00 mm
- net /BLANK: track 40.9 -> 0.00 mm
- net /H_PWM_N: track 40.6 -> 0.00 mm
- net /MOSI: track 39.2 -> 0.00 mm
- net Net-(CN7-Pad14): track 38.8 -> 0.00 mm
- net /EN24: track 32.8 -> 0.00 mm, vias 1 -> 0
- net /D8: track 32.1 -> 0.00 mm
- net /STATUS: track 29.2 -> 0.00 mm
- net /D0: track 27.8 -> 0.00 mm
- net /D7: track 26.4 -> 0.00 mm
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Other:
- board size 69.9 x 74.9 mm -> 99.1 x 71.1 mm
- board text added: "MOSI"
- board text added: "SCK"
- board text removed: "A"
- board text removed: "SPI1_MOSI"
- board text removed: "SPI1_SCK"

Commit message: Revert "Changed from Nucleo to RPi Pico"
This reverts commit 16e9e4a1a83ee259be72a8795d021f70ac3e2adc.
Parts:
- removed U5: Pico, LOCAL_LIB:RPi_Pico_SMD_TH
- added CN10: PPPC192LFBN-RC, Connector_PinSocket_2.54mm:PinSocket_2x19_P2.54mm_Vertical, B.Cu at (180.3, 61.0)
- added CN7: PPPC192LFBN-RC, Connector_PinSocket_2.54mm:PinSocket_2x19_P2.54mm_Vertical, B.Cu at (119.4, 61.0)
- added R1: 1k, Capacitor_SMD:C_0603_1608Metric_Pad1.08x0.95mm_HandSolder, F.Cu at (130.8, 48.3)
- D1, D2: footprint Diode_SMD:D_0603_1608Metric_Pad1.05x0.95mm_HandSolder -> Capacitor_SMD:C_0603_1608Metric_Pad1.08x0.95mm_HandSolder
- D3: value D_Schottky -> LED; footprint Diode_SMD:D_0603_1608Metric_Pad1.05x0.95mm_HandSolder -> LED_THT:LED_D4.0mm
- SW1: value SW_MEC_5E -> SW
- moved SW1 83.5 mm to (118.7, 40.9)
- moved TP3 77.6 mm to (182.9, 45.7)
- moved J1 49.7 mm to (171.5, 106.7), turned to 180 degrees
- moved TP6 37.1 mm to (176.5, 72.4)
- moved C1 25.4 mm to (170.2, 39.4), turned to 90 degrees
- moved L1 24.4 mm to (175.8, 40.6)
- moved TP9 23.2 mm to (127.0, 63.5)
- moved TP4 21.8 mm to (135.9, 57.1)
- moved JP4 20.7 mm to (170.2, 47.0)
- moved JP3 20.3 mm to (165.7, 48.3)
- moved JP1 16.2 mm to (175.9, 51.4)
- moved TP5 15.5 mm to (176.5, 104.1)
- moved U3 15.5 mm to (175.3, 48.3)
- moved C6 15.4 mm to (181.6, 53.4), turned to -90 degrees
- moved JP2 14.7 mm to (151.8, 61.0)
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Connections:
- net /CHARGE_P_PWM renamed /TIM2_CH1
- net /H_PWM_N renamed /TIM1_CH1N
- net /H_PWM_P renamed /TIM1_CH1
- net /MOSI renamed /SPI1_MOSI
- net /SCK renamed /SPI1_SCK
- D3 pad 2: +BATT -> /STATUS
- SW1 pad 1: Net-(SW1-Pad1) -> GND
- SW1 pad 2: Net-(SW1-Pad1) -> GND
- SW1 pad 3: GND -> Net-(CN7-Pad14)
- SW1 pad 4: GND -> Net-(CN7-Pad14)
- U1 pad 20: unconnected-(U1-Pad20) -> /Seg_a
- U1 pad 25: /D0 -> /D8
- U1 pad 26: /Seg_b -> /Seg_g
- U1 pad 27: /D1 -> /D7
- U1 pad 3: /Seg_a -> unconnected-(U1-Pad3)
- U1 pad 30: /D2 -> /Seg_f
- U1 pad 32: /DP -> /Seg_e
- U1 pad 33: /D3 -> /D5
- U1 pad 34: /Seg_d -> /D4
- U1 pad 35: /D4 -> /Seg_d
- U1 pad 36: /D5 -> /D3
- U1 pad 37: /Seg_e -> /DP
- U1 pad 38: /Seg_c -> /D2
- U1 pad 39: /Seg_f -> /Seg_c
- U1 pad 40: /D7 -> /D1
- U1 pad 41: /Seg_g -> /Seg_b
- U1 pad 42: /D8 -> /D0
Routing:
- net /TIM2_CH1: track 0.00 -> 62.1 mm
- net /SPI1_SCK: track 0.00 -> 52.2 mm
- net /TIM1_CH1: track 0.00 -> 47.8 mm
- net /LOAD: track 0.00 -> 46.9 mm
- net +BATT: track 0.00 -> 42.7 mm
- net /Seg_a: track 0.00 -> 41.4 mm
- net /BLANK: track 0.00 -> 40.9 mm
- net /TIM1_CH1N: track 0.00 -> 40.6 mm
- net /SPI1_MOSI: track 0.00 -> 39.2 mm
- net Net-(CN7-Pad14): track 0.00 -> 38.8 mm
- net /EN24: track 0.00 -> 32.8 mm, vias 0 -> 1
- net /D8: track 0.00 -> 32.1 mm
- net /STATUS: track 0.00 -> 29.2 mm
- net /D0: track 0.00 -> 27.8 mm
- net /D7: track 0.00 -> 26.4 mm
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Other:
- board size 99.1 x 71.1 mm -> 69.9 x 74.9 mm
- board text added: "A"
- board text added: "SPI1_MOSI"
- board text added: "SPI1_SCK"
- board text removed: "MOSI"
- board text removed: "SCK"

Commit message: Gerber file generated
Parts:
- moved JP2 8.28 mm to (144.8, 65.4)
Connections:
- U1 pad 25: /D8 -> /D0
- U1 pad 26: /Seg_g -> /Seg_b
- U1 pad 27: /D7 -> /D1
- U1 pad 30: /Seg_f -> /Seg_c
- U1 pad 31: /D6 -> /D2
- U1 pad 32: /Seg_e -> /DP
- U1 pad 33: /D5 -> /D3
- U1 pad 34: /D4 -> /Seg_d
- U1 pad 35: /Seg_d -> /D4
- U1 pad 36: /D3 -> /D5
- U1 pad 37: /DP -> /Seg_e
- U1 pad 38: /D2 -> /D6
- U1 pad 39: /Seg_c -> /Seg_f
- U1 pad 40: /D1 -> /D7
- U1 pad 41: /Seg_b -> /Seg_g
- U1 pad 42: /D0 -> /D8
Routing:
- net /Seg_b: track 25.3 -> 46.3 mm
- net /D0: track 27.8 -> 45.4 mm
- net /D1: track 24.2 -> 40.4 mm
- net /Seg_c: track 20.6 -> 36.5 mm
- net /Seg_g: track 25.5 -> 39.4 mm
- net /D8: track 32.1 -> 44.9 mm
- net /D6: track 19.4 -> 31.5 mm
- net /D7: track 26.4 -> 37.5 mm
- net +24V: track 25.4 -> 15.8 mm
- net /D5: track 18.5 -> 28.0 mm
- net /Seg_f: track 24.0 -> 32.7 mm
- net /SPI1_SCK: track 52.2 -> 60.1 mm, vias 0 -> 2
- net /DP: track 19.6 -> 26.2 mm
- net Net-(C9-Pad1): track 18.0 -> 24.5 mm, vias 0 -> 1
- net /Seg_d: track 18.5 -> 24.2 mm, vias 0 -> 1
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Other:
- rule pad_to_mask_clearance: 0.051 -> 0
