File: Akashi-11.kicad_sch (KiCad schematic)
At the start: 43 parts, among them J1 Conn_02x20_Odd_Even, SW1 SW_MEC_5E, U1 MAX6934AQH+D, U2 MAX4719EUB+, U3 TPS613221ADBV, U4 TLV61046ADB, U5 Pico

Commit message: Revert "Changed from Nucleo to RPi Pico"
This reverts commit 16e9e4a1a83ee259be72a8795d021f70ac3e2adc.
Parts:
- removed D3: D_Schottky, Diode_SMD:D_0603_1608Metric_Pad1.05x0.95mm_HandSolder, symbol Device:D_Schottky
- removed SW1: SW_MEC_5E, Button_Switch_THT:SW_TH_Tactile_Omron_B3F-10xx, symbol Switch:SW_MEC_5E
- removed U5: Pico, RPi_Pico:RPi_Pico_SMD_TH, symbol RPI_PICO:Pico
- added CN10, CN7: PPPC192LFBN-RC, Connector_PinSocket_2.54mm:PinSocket_2x19_P2.54mm_Vertical, symbol Connector_Generic:Conn_02x19_Odd_Even
- added D3: LED, LED_THT:LED_D4.0mm, symbol Device:LED
- added R1: 1k, Capacitor_SMD:C_0603_1608Metric_Pad1.08x0.95mm_HandSolder, symbol Device:R
- added SW1: SW, Button_Switch_THT:SW_TH_Tactile_Omron_B3F-10xx, symbol Switch:SW_MEC_5G
- D1, D2: footprint Diode_SMD:D_0603_1608Metric_Pad1.05x0.95mm_HandSolder -> Capacitor_SMD:C_0603_1608Metric_Pad1.08x0.95mm_HandSolder
Connections:
- net +3V3: now also CN7.12 (Pin_12), CN7.16 (Pin_16)
- net BLANK: now also CN7.3 (Pin_3)
- net D0: now also U1.42 (OUT0); no longer U1.25 (OUT15)
- net D1: now also U1.40 (OUT2); no longer U1.27 (OUT13)
- net D2: now also U1.38 (OUT4); no longer U1.30 (OUT12)
- net D3: now also U1.36 (OUT6); no longer U1.33 (OUT9)
- net D4: now also U1.34 (OUT8); no longer U1.35 (OUT7)
- net D5: now also U1.33 (OUT9); no longer U1.36 (OUT6)
- net D7: now also U1.27 (OUT13); no longer U1.40 (OUT2)
- net D8: now also U1.25 (OUT15); no longer U1.42 (OUT0)
- net DP: now also U1.37 (OUT5); no longer U1.32 (OUT10)
- net EN24: now also CN7.2 (Pin_2)
- net GND: now also CN10.20 (Pin_20), CN10.32 (Pin_32), CN10.9 (Pin_9), CN7.19 (Pin_19), CN7.20 (Pin_20), CN7.22 (Pin_22), CN7.8 (Pin_8), R1.2, SW1.1 (A), SW1.2 (A)
- net KD0: now also CN10.11 (Pin_11)
- net KD1: now also CN10.13 (Pin_13)
- net KD2: now also CN10.16 (Pin_16)
- net KD3: now also CN10.17 (Pin_17)
- net KD4: now also CN10.19 (Pin_19)
- net KD5: now also CN10.22 (Pin_22)
- net KD6: now also CN10.24 (Pin_24)
- net KD7: now also CN10.25 (Pin_25)
- net KD8: now also CN10.27 (Pin_27)
- net KEY1: now also CN10.33 (Pin_33)
- net KEY2: now also CN10.31 (Pin_31)
- net KEY3: now also CN10.29 (Pin_29)
- net LOAD: now also CN7.1 (Pin_1)
- net Seg_a: now also U1.20 (OUT16); no longer U1.3 (OUT31)
- net Seg_b: now also U1.41 (OUT1); no longer U1.26 (OUT14)
- net Seg_c: now also U1.39 (OUT3); no longer U1.38 (OUT4)
- net Seg_d: now also U1.35 (OUT7); no longer U1.34 (OUT8)
- net Seg_e: now also U1.32 (OUT10); no longer U1.37 (OUT5)
- net Seg_f: now also U1.30 (OUT12); no longer U1.39 (OUT3)
- net Seg_g: now also U1.26 (OUT14); no longer U1.41 (OUT1)
- net CHARGE_P_PWM renamed TIM2_CH1
- net TIM2_CH1: now also CN10.21 (Pin_21)
- net H_PWM_N renamed TIM1_CH1N
- net TIM1_CH1N: now also CN10.15 (Pin_15)
- net H_PWM_P renamed TIM1_CH1
- net TIM1_CH1: now also CN10.23 (Pin_23)
- net MOSI renamed SPI1_MOSI
- net SPI1_MOSI: now also CN10.12 (Pin_12)
- net SCK renamed SPI1_SCK
- net SPI1_SCK: now also CN10.36 (Pin_36)
- new net: CN7.14 (Pin_14), SW1.3 (B), SW1.4 (B)
- new net: D3.1 (K), R1.1
- new net STATUS: CN7.4 (Pin_4), D3.2 (A)
- no-connect marks 36 -> 68
Other:
- note added: "PA10"
- note added: "PA12"
- note added: "PA5"
- note added: "PA6"
- note added: "PA7"
- note added: "PA8"
- note added: "PA9"
- note added: "PB0"
- note added: "PB14"
- note added: "PB2"
- note added: "PB3"
- note added: "PB4"
- note added: "PB5"
- note added: "PB6"
- note added: "PC1"
- note added: "PC10"
- note added: "PC12"
- note added: "PC7"
- note added: "PD8"
- note added: "STATUS"
- moved on the sheet: C3, C5, C8, J1, JP3, JP4, TP2, U1

Commit message: Gerber file generated
Parts:
- C6: value UZG0J220MCL1GB -> 22u
- C9: value UZG1H100MCL1GB -> 10u
- L1: value LQH5BPN4R7N38L -> 4.7u
- L2: value LQH5BPN100M38L -> 10u
Connections:
- net D0: now also U1.25 (OUT15); no longer U1.42 (OUT0)
- net D1: now also U1.27 (OUT13); no longer U1.40 (OUT2)
- net D2: now also U1.31 (OUT11); no longer U1.38 (OUT4)
- net D3: now also U1.33 (OUT9); no longer U1.36 (OUT6)
- net D4: now also U1.35 (OUT7); no longer U1.34 (OUT8)
- net D5: now also U1.36 (OUT6); no longer U1.33 (OUT9)
- net D6: now also U1.38 (OUT4); no longer U1.31 (OUT11)
- net D7: now also U1.40 (OUT2); no longer U1.27 (OUT13)
- net D8: now also U1.42 (OUT0); no longer U1.25 (OUT15)
- net DP: now also U1.32 (OUT10); no longer U1.37 (OUT5)
- net Seg_b: now also U1.26 (OUT14); no longer U1.41 (OUT1)
- net Seg_c: now also U1.30 (OUT12); no longer U1.39 (OUT3)
- net Seg_d: now also U1.34 (OUT8); no longer U1.35 (OUT7)
- net Seg_e: now also U1.37 (OUT5); no longer U1.32 (OUT10)
- net Seg_f: now also U1.39 (OUT3); no longer U1.30 (OUT12)
- net Seg_g: now also U1.41 (OUT1); no longer U1.26 (OUT14)
Changed lines of the file:
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@@
     (effects (font (size 1.27 1.27)) (justify left bottom))
   )
-  (label "DP" (at 142.24 54.61 0)
+  (label "DP" (at 142.24 67.31 0)
     (effects (font (size 1.27 1.27)) (justify left bottom))
   )
@@
     (effects (font (size 1.27 1.27)) (justify left bottom))
   )
-  (label "Seg_d" (at 142.24 59.69 0)
-    (effects (font (size 1.27 1.27)) (justify left bottom))
-  )
-  (label "Seg_b" (at 142.24 44.45 0)
+  (label "Seg_d" (at 142.24 62.23 0)
+    (effects (font (size 1.27 1.27)) (justify left bottom))
+  )
+  (label "Seg_b" (at 142.24 82.55 0)
     (effects (font (size 1.27 1.27)) (justify left bottom))
   )
@@
     (effects (font (size 1.27 1.27)) (justify left bottom))
   )
-  (label "Seg_e" (at 142.24 67.31 0)
+  (label "Seg_e" (at 142.24 54.61 0)
     (effects (font (size 1.27 1.27)) (justify left bottom))
   )
@@
     (effects (font (size 1.27 1.27)) (justify left bottom))
   )
-  (label "D7" (at 142.24 80.01 0)
+  (label "D7" (at 142.24 46.99 0)
     (effects (font (size 1.27 1.27)) (justify left bottom))
   )
@@
     (effects (font (size 1.27 1.27)) (justify left bottom))
   )
-  (label "D1" (at 142.24 46.99 0)
-    (effects (font (size 1.27 1.27)) (justify left bottom))
-  )
-  (label "D8" (at 142.24 85.09 0)
+  (label "D1" (at 142.24 80.01 0)
+    (effects (font (size 1.27 1.27)) (justify left bottom))
+  )
+  (label "D8" (at 142.24 41.91 0)
     (effects (font (size 1.27 1.27)) (justify left bottom))
   )
@@
     (effects (font (size 1.27 1.27)) (justify left bottom))
   )
-  (label "D2" (at 142.24 52.07 0)
+  (label "D2" (at 142.24 69.85 0)
     (effects (font (size 1.27 1.27)) (justify left bottom))
   )
@@
     (effects (font (size 1.27 1.27)) (justify left bottom))
   )
-  (label "D6" (at 142.24 69.85 0)
+  (label "D6" (at 142.24 52.07 0)
     (effects (font (size 1.27 1.27)) (justify left bottom))
   )
@@
     (effects (font (size 1.27 1.27)) (justify left bottom))
   )
-  (label "Seg_g" (at 142.24 82.55 0)
+  (label "Seg_g" (at 142.24 44.45 0)
     (effects (font (size 1.27 1.27)) (justify left bottom))
   )
@@
     (effects (font (size 1.27 1.27)) (justify left bottom))
   )
-  (label "Seg_f" (at 142.24 72.39 0)
+  (label "Seg_f" (at 142.24 49.53 0)
     (effects (font (size 1.27 1.27)) (justify left bottom))
   )
@@
     (effects (font (size 1.27 1.27)) (justify left bottom))
   )
-  (label "D4" (at 142.24 62.23 0)
+  (label "D4" (at 142.24 59.69 0)
     (effects (font (size 1.27 1.27)) (justify left bottom))
   )
@@
     (effects (font (size 1.27 1.27)) (justify left bottom))
   )
-  (label "Seg_c" (at 142.24 49.53 0)
+  (label "Seg_c" (at 142.24 72.39 0)
     (effects (font (size 1.27 1.27)) (justify left bottom))
   )
@@
     (effects (font (size 1.27 1.27)) (justify left bottom))
   )
-  (label "D0" (at 142.24 41.91 0)
+  (label "D0" (at 142.24 85.09 0)
     (effects (font (size 1.27 1.27)) (justify left bottom))
   )
@@
     (effects (font (size 1.27 1.27)) (justify left bottom))
   )
-  (label "D5" (at 142.24 64.77 0)
-    (effects (font (size 1.27 1.27)) (justify left bottom))
-  )
-  (label "D3" (at 142.24 57.15 0)
+  (label "D5" (at 142.24 57.15 0)
+    (effects (font (size 1.27 1.27)) (justify left bottom))
+  )
+  (label "D3" (at 142.24 64.77 0)
     (effects (font (size 1.27 1.27)) (justify left bottom))
   )
@@
     (in_bom yes) (on_board yes) (fields_autoplaced)
     (property "Reference" "L2" (id 0) (at 226.06 113.9022 90))
-    (property "Value" "LQH5BPN100M38L" (id 1) (at 226.06 116.4391 90))
+    (property "Value" "10u" (id 1) (at 226.06 116.4391 90))
     (property "Footprint" "LOCAL_LIB:LQH5BPN100M38L" (id 2) (at 226.06 118.11 0)
       (effects (font (size 1.27 1.27)) hide)
     )
-    (property "Datasheet" "~" (id 3) (at 226.06 118.11 0)
+    (property "Datasheet" "LQH5BPN100M38L" (id 3) (at 226.06 118.11 0)
       (effects (font (size 1.27 1.27)) hide)
     )
@@
       (effects (font (size 1.27 1.27)) (justify left))
     )
-    (property "Value" "UZG0J220MCL1GB" (id 1) (at 72.009 172.6061 0)
+    (property "Value" "22u" (id 1) (at 72.009 172.6061 0)
       (effects (font (size 1.27 1.27)) (justify left))
     )
@@
       (effects (font (size 1.27 1.27)) hide)
     )
-    (property "Datasheet" "~" (id 3) (at 69.85 171.45 0)
+    (property "Datasheet" "UZG0J220MCL1GB" (id 3) (at 69.85 171.45 0)
       (effects (font (size 1.27 1.27)) hide)
     )
@@
       (effects (font (size 1.27 1.27)) (justify left))
     )
-    (property "Value" "UZG1H100MCL1GB" (id 1) (at 251.079 145.9361 0)
+    (property "Value" "10u" (id 1) (at 251.079 145.9361 0)
       (effects (font (size 1.27 1.27)) (justify left))
     )
@@
       (effects (font (size 1.27 1.27)) hide)
     )
-    (property "Datasheet" "~" (id 3) (at 248.92 144.78 0)
+    (property "Datasheet" "UZG1H100MCL1GB" (id 3) (at 248.92 144.78 0)
       (effects (font (size 1.27 1.27)) hide)
     )
@@
     (in_bom yes) (on_board yes)
     (property "Reference" "L1" (id 0) (at 36.83 160.8922 90))
-    (property "Value" "LQH5BPN4R7N38L" (id 1) (at 36.83 167.64 90))
+    (property "Value" "4.7u" (id 1) (at 36.83 167.64 90))
     (property "Footprint" "LOCAL_LIB:LQH5BPN100M38L" (id 2) (at 36.83 165.1 0)
       (effects (font (size 1.27 1.27)) hide)
     )
-    (property "Datasheet" "~" (id 3) (at 36.83 165.1 0)
+    (property "Datasheet" "LQH5BPN4R7N38L" (id 3) (at 36.83 165.1 0)
       (effects (font (size 1.27 1.27)) hide)
     )
@@
     )
     (path "/746d5d6e-d183-4a43-98fc-0910c3a56939"
-      (reference "C6") (unit 1) (value "UZG0J220MCL1GB") (footprint "Capacitor_SMD:CP_Elec_6.3x3")
+      (reference "C6") (unit 1) (value "22u") (footprint "Capacitor_SMD:CP_Elec_6.3x3")
     )
     (path "/03f09313-6917-4cb7-9358-3b4f9e115ab2"
@@
     )
     (path "/ce4a2bdc-5956-467a-becf-ee6582a3ff8f"
-      (reference "C9") (unit 1) (value "UZG1H100MCL1GB") (footprint "Capacitor_SMD:CP_Elec_4x3.9")
+      (reference "C9") (unit 1) (value "10u") (footprint "Capacitor_SMD:CP_Elec_4x3.9")
     )
     (path "/00000000-0000-0000-0000-00005c96bbda"
@@
     )
     (path "/f2deddfd-89b8-4596-90ac-4edc0864ba22"
-      (reference "L1") (unit 1) (value "LQH5BPN4R7N38L") (footprint "LOCAL_LIB:LQH5BPN100M38L")
+      (reference "L1") (unit 1) (value "4.7u") (footprint "LOCAL_LIB:LQH5BPN100M38L")
     )
     (path "/71d170b5-c318-465b-b133-162877591a12"
-      (reference "L2") (unit 1) (value "LQH5BPN100M38L") (footprint "LOCAL_LIB:LQH5BPN100M38L")
+      (reference "L2") (unit 1) (value "10u") (footprint "LOCAL_LIB:LQH5BPN100M38L")
     )
     (path "/f9dedb24-0217-47a0-b3d0-1a79d739bcb2"

Commit message: Change signal name from TIM2_CH1 to TIM1_CH2
Fixed typo. The layout is not changed.
The sylkscreen of the singal is still wrong.
Parts:
- R2: value 61.9 -> 61.9k
- R3: value 2.15 -> 2.15k
Connections:
- net TIM2_CH1 renamed TIM1_CH2
Changed lines of the file:
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@@
     (effects (font (size 1.27 1.27)) (justify left bottom))
   )
-  (label "TIM2_CH1" (at 113.03 152.4 0)
+  (label "TIM1_CH2" (at 113.03 152.4 0)
     (effects (font (size 1.27 1.27)) (justify left bottom))
   )
@@
     (effects (font (size 1.27 1.27)) (justify left bottom))
   )
-  (label "TIM2_CH1" (at 231.14 64.77 0)
+  (label "TIM1_CH2" (at 231.14 64.77 0)
     (effects (font (size 1.27 1.27)) (justify left bottom))
   )
@@
       (effects (font (size 1.27 1.27)) (justify left))
     )
-    (property "Value" "2.15" (id 1) (at 243.078 151.5622 0)
+    (property "Value" "2.15k" (id 1) (at 243.078 151.5622 0)
       (effects (font (size 1.27 1.27)) (justify left))
     )
@@
       (effects (font (size 1.27 1.27)) (justify left))
     )
-    (property "Value" "61.9" (id 1) (at 243.078 138.8622 0)
+    (property "Value" "61.9k" (id 1) (at 243.078 138.8622 0)
       (effects (font (size 1.27 1.27)) (justify left))
     )
@@
     )
     (path "/680642e7-76ab-4f46-85b1-7e8240ef7d1b"
-      (reference "R2") (unit 1) (value "61.9") (footprint "Capacitor_SMD:C_0603_1608Metric_Pad1.08x0.95mm_HandSolder")
+      (reference "R2") (unit 1) (value "61.9k") (footprint "Capacitor_SMD:C_0603_1608Metric_Pad1.08x0.95mm_HandSolder")
     )
     (path "/13bc741c-df8f-46cd-81b6-34ab4aece211"
-      (reference "R3") (unit 1) (value "2.15") (footprint "Capacitor_SMD:C_0603_1608Metric_Pad1.08x0.95mm_HandSolder")
+      (reference "R3") (unit 1) (value "2.15k") (footprint "Capacitor_SMD:C_0603_1608Metric_Pad1.08x0.95mm_HandSolder")
     )
     (path "/aa7e72ca-4dfc-42eb-9354-239397f2ab9c"
